File: eagle/MFOS_VCO_edge.sch (EAGLE design)
At the start: 110 parts, among them IC1 TL072P, IC2 LM394N, IC3 TL072P, IC4 TL072P, IC5 TL072P, IC6 TL072P, IC7 LM13700N, U1 2N5457, U2 POWER

Commit message: flexible trimmers and grounded air outputs and connector for PWM pot
Parts:
- removed CV1: 22-23-2021, con-molex:22-23-2021
- removed HIGH_FREQ_TRIM, SINE_SHAPE: 100k, pot:TRIM_US-B64Y
- removed R21, TRI_OFFSET: 10k, pot:TRIM_US-B64Y
- removed R36: 100k, pot:3RP/1610N
- removed SCALE_TRIM: 100R, pot:TRIM_US-B64Y
- removed SINE_LEVEL: 1M, pot:TRIM_US-B64Y
- added CV3: (no value), con-phoenix-254:MPT2
- added HF_TRIM, SINE: 100k, pot:TRIM_US-B64W
- added PWM_POT: 100k, con-phoenix-254:MPT3
- added RAMP_OFF, TRI_OFF: 10k, pot:TRIM_US-B64W
- added SCALE: 100R, pot:TRIM_US-B64W
- added SINE_LEV: 1M, pot:TRIM_US-B64W
- C11: value 0.1uF -> 100n
- C8: value .005uF -> 5nF PSA
- C9: value .001uF -> 1n
- CV2: value 22-23-2021 -> (none); device con-molex:22-23-2021 -> con-phoenix-254:MPT2
- PWM, SQR, TRI: value LSP10 -> (none); device solpad:LSP10 -> con-phoenix-254:MPT2
- R23: device rcl:R-US_0207/10 -> rcl:R-US_0207/7
- SINE_BIAS: device pot:TRIM_US-B64Y -> pot:TRIM_US-B64W
- renumbered R12-TEMPCO to TEMPCO
Connections:
- net +12V: now also SINE_LEV.E; no longer SINE_LEVEL.E
- net GND: now also CV2-2.1, CV3-2.1, PWM-2.1, RAMP_OFF.A, SQR-2.1, TRI-2.1, TRI_OFF.A; no longer CV1-2.S, CV2-2.S, R21.A, TRI_OFFSET.A
- net N$14: now also HF_TRIM.E, HF_TRIM.S; no longer HIGH_FREQ_TRIM.E, HIGH_FREQ_TRIM.S
- net N$16: now also HF_TRIM.A; no longer HIGH_FREQ_TRIM.A
- net N$18: now also CV2-1.1; no longer CV1-1.S
- net N$19: now also CV3-1.1; no longer CV2-1.S
- net N$27: now also RAMP_OFF.E; no longer R21.E
- net N$28: now also RAMP_OFF.S; no longer R21.S
- net N$46: now also SINE.E; no longer SINE_SHAPE.E
- net N$47: now also TRI-1.1; no longer TRI.MP
- net N$48: now also TRI_OFF.E; no longer TRI_OFFSET.E
- net N$49: now also TRI_OFF.S; no longer TRI_OFFSET.S
- net N$52: now also PWM_POT-1.1; no longer R36.E
- net N$53: now also PWM_POT-3.1; no longer R36.A
- net N$54: now also PWM-1.1; no longer PWM.MP
- net N$57: now also SQR-1.1; no longer SQR.MP
- net N$59: now also PWM_POT-2.1; no longer R36.S
- net N$60: now also SINE.A, SINE.S; no longer SINE_SHAPE.A, SINE_SHAPE.S
- net N$64: now also SINE_LEV.A, SINE_LEV.S; no longer SINE_LEVEL.A, SINE_LEVEL.S
- net N$7: now also SCALE.A; no longer SCALE_TRIM.A
- net N$8: now also SCALE.S; no longer SCALE_TRIM.S
- net N$9: now also SCALE.E; no longer SCALE_TRIM.E
Other:
- moved on the sheet: CV_IN, R11
