File: eagle/MFOS_VCO_edge.sch (EAGLE design)
At the start: 110 parts, among them IC1 TL072P, IC2 LM394N, IC3 TL072P, IC4 TL072P, IC5 TL072P, IC6 TL072P, IC7 LM13700N, U1 2N5457, U2 POWER

Commit message: changes
Parts:
- C14: value 0.002uF -> 2nF
- C7: value 0.1uF -> 100nF
Changed lines of the file:
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@@
 <part name="P+6" library="supply1" deviceset="+12V" device=""/>
 <part name="GND9" library="supply1" deviceset="GND" device=""/>
-<part name="C7" library="rcl" deviceset="C-US" device="050-024X044" value="0.1uF"/>
+<part name="C7" library="rcl" deviceset="C-US" device="050-024X044" value="100nF"/>
 <part name="R22" library="rcl" deviceset="R-US_" device="0207/7" value="10k"/>
 <part name="GND10" library="supply1" deviceset="GND" device=""/>
@@
 <part name="GND21" library="supply1" deviceset="GND" device=""/>
 <part name="R18" library="rcl" deviceset="R-US_" device="0207/7" value="20k"/>
-<part name="C14" library="rcl" deviceset="C-US" device="050-030X075" value="0.002uF"/>
+<part name="C14" library="rcl" deviceset="C-US" device="050-030X075" value="2nF"/>
 <part name="P-9" library="supply1" deviceset="-12V" device=""/>
 <part name="C15" library="rcl" deviceset="CPOL-US" device="B45181A" value="1uF tant"/>
