File: eagle/MFOS_VCO_edge.brd (EAGLE design)
At the start: 97.8 x 78.7 mm, 110 parts, among them IC1 TL072P, IC2 LM394N, IC3 TL072P, IC4 TL072P, IC5 TL072P, IC6 TL072P, IC7 LM13700N, U1 2N5457, U2 POWER

Commit message: changes
Parts:
- C14: value 0.002uF -> 2nF
- C7: value 0.1uF -> 100nF
- moved R4 21.1 mm to (51.8, 75.9), turned to 0 degrees
- moved R10 4.77 mm to (59.4, 21.5), turned to 90 degrees
- moved R11 3.98 mm to (62.5, 21.7), turned to 90 degrees
- moved R17 2.81 mm to (49.7, 30.5), turned to 90 degrees
- moved R9 2.69 mm to (56.1, 21.5), turned to 90 degrees
- moved R29 1.27 mm to (32.9, 46.5)
- moved R30 1.27 mm to (28.8, 49.8)
- moved R32 0.92 mm to (17.5, 30.2)
- moved R26 0.25 mm to (18.5, 37.0)
- moved U1 0.25 mm to (16.9, 27.4)
Routing:
- net N$9: track 46.0 -> 88.5 mm
- net N$46: track 64.5 -> 24.8 mm
- net +12V: track 226.3 -> 251.3 mm, vias 1 -> 0
- net N$49: track 55.2 -> 72.5 mm, vias 1 -> 2
- net N$13: track 100.2 -> 88.0 mm
- net N$56: track 74.5 -> 63.0 mm, vias 0 -> 1
- net N$66: track 74.5 -> 63.2 mm, vias 2 -> 0
- net N$10: track 104.5 -> 114.8 mm
- net N$15: track 10.5 -> 3.83 mm
- net N$18: track 14.1 -> 7.69 mm
- net N$21: track 32.5 -> 26.8 mm
- net GND: track 433.1 -> 427.8 mm
- net N$7: track 17.2 -> 22.3 mm
- net -12V: track 250.8 -> 247.2 mm, vias 0 -> 1
- net N$45: track 69.0 -> 65.5 mm
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